Commit message: Spawning in Rviz and Gazebo

File: diff_drive/ddrive.gazebo.xacro (robot description, xacro)
@@ -1,11 +1,14 @@
-<robot name="Diff Drive" xmlns:xacro="http://www.ros.org/wiki/xacro">
+<robot name="DiffDrive" xmlns:xacro="http://www.ros.org/wiki/xacro">
     <gazebo reference="body">
-        <material> material Gazebo/TurquoiseGlow </material>
+        <material>Gazebo/Yellow</material>
     </gazebo>
     <gazebo reference="right_wheel">
-        <material> material Gazebo/LightBlueLaser </material>
+        <material>Gazebo/Blue</material>
     </gazebo>
     <gazebo reference="left_wheel">
-        <material>material Gazebo/Bricks </material>
+        <material>Gazebo/Blue</material>
+    </gazebo>
+    <gazebo reference="caster">
+        <material>Gazebo/Blue</material>
     </gazebo>
 </robot>

File: diff_drive/ddrive.urdf.xacro (robot description, xacro)
@@ -1,4 +1,4 @@
 <?xml version = "1.0"?>
-<robot name="Diff Drive" xmlns:xacro="http://www.ros.org/wiki/xacro">
+<robot name="DiffDrive" xmlns:xacro="http://www.ros.org/wiki/xacro">
 <xacro:include filename="ddrive.gazebo.xacro"/>
 <xacro:property name="robot_params" value = "$(find diff_drive)/config/robot_params.yaml" />
@@ -11,22 +11,5 @@
 <xacro:property name="l" value="${params['wheel_l']}"/>
 <xacro:property name="wheel_m" value="${params['wheel_mass']}"/>
-<link name="base">
-    <visual>
-        <origin xyz="0 0 0" rpy="0 0 0"/>
-        <mass value="1"/>
-        <geometry>
-            <box size=".001 .001 .001" />
-        </geometry>
-        <material name="trans_mat">
-            <color rgba="0 0 0 0" />
-        </material>
-    </visual>
-</link>
-<joint name="fixed" type="fixed">
-  <parent link="base" />
-  <child link="body" />
-  <axis xyz = "0 0 1" />
-  <origin xyz="0 0 0" rpy="0 0 0" />
-</joint>
+<link name="base" />
 <link name="body">
     <inertial>
@@ -51,18 +34,12 @@
   </collision>
 </link>
-<joint name="joint1" type="continuous">
-  <parent link="body" />
-  <child link="right_wheel" />
-  <axis xyz = "0 0 1" />
-  <origin xyz="0 ${Y/2} ${Z/2}" rpy="0 0 0" />
-</joint>
 <link name="right_wheel">
-  <visual>
    <inertial>
-     <origin xyz="0 0 ${l/2}" rpy="0 0 0"/>
+     <origin xyz="0 0 ${-1*l}" rpy="0 0 0"/>
      <mass value="${wheel_m}"/>
      <inertia ixx="1"  ixy="1"  ixz="1" iyy="1" iyz="1" izz="1" />
    </inertial>
-   <origin xyz="0 0 ${l/2}" rpy="0 0 0"/>
+  <visual>
+   <origin xyz="0 0 ${-1*l}" rpy="0 0 0"/>
    <geometry>
      <cylinder radius="${r}" length="${l}" />
@@ -73,5 +50,5 @@
   </visual>
   <collision>
-    <origin xyz="0 0 ${l/2}" rpy="0 0 0"/>
+   <origin xyz="0 0 ${-1*l}" rpy="0 0 0"/>
    <geometry>
      <cylinder radius="${r}" length="${l}" />
@@ -79,18 +56,12 @@
   </collision>
 </link>
-<joint name="joint2" type="continuous">
-  <parent link="body" />
-  <child link="left_wheel" />
-  <axis xyz = "0 0 1" />
-  <origin xyz="0 ${Y/2} ${-Z/2}" rpy="0 0 0" />
-</joint>
 <link name="left_wheel">
-  <visual>
    <inertial>
-     <origin xyz=" 0 0 ${-1*l/2}" rpy="0 0 0"/>
+     <origin xyz=" 0 0 ${l/2}" rpy="0 0 0"/>
      <mass value="${wheel_m}"/>
      <inertia ixx="1"  ixy="1"  ixz="1" iyy="1" iyz="1" izz="1" />
    </inertial>
-   <origin xyz=" 0 0 ${-1*l/2}" rpy="0 0 0"/>
+  <visual>
+   <origin xyz=" 0 0 ${l/2}" rpy="0 0 0"/>
    <geometry>
      <cylinder radius="${r}" length="${l}" />
@@ -101,5 +72,5 @@
   </visual>
   <collision>
-     <origin xyz=" 0 0 ${-1*l/2}" rpy="0 0 0"/>
+     <origin xyz=" 0 0 ${l/2}" rpy="0 0 0"/>
    <geometry>
     <cylinder radius="${r}" length="${l}" />
@@ -107,3 +78,47 @@
   </collision>
 </link>
+<link name="caster">
+   <inertial>
+     <origin xyz=" 0 0 0" rpy="0 0 0"/>
+     <mass value="${wheel_m}"/>
+     <inertia ixx="1"  ixy="1"  ixz="1" iyy="1" iyz="1" izz="1" />
+   </inertial>
+  <visual>
+   <origin xyz=" 0 0 0" rpy="0 0 0"/>
+   <geometry>
+     <cylinder radius="${Z}" length="${l}" />
+   </geometry>
+     <material name="cyan_mat">
+         <color rgba="0 1 1 1" />
+     </material>
+  </visual>
+  <collision>
+     <origin xyz=" 0 0 0" rpy="0 0 0"/>
+   <geometry>
+    <cylinder radius="${r}" length="${l}" />
+   </geometry>
+  </collision>
+</link>
+<joint name="fixed" type="fixed">
+  <parent link="base" />
+  <child link="body" />
+  <origin xyz="0 0 0" rpy="0 0 0" />
+</joint>
+<joint name="joint1" type="continuous">
+  <parent link="body" />
+  <child link="right_wheel" />
+  <axis xyz = "0 0 1" />
+  <origin xyz="${X/2} ${Y/2} 0" rpy="0 -1.57 0" />
+</joint>
+<joint name="joint2" type="continuous">
+  <parent link="body" />
+  <child link="left_wheel" />
+  <axis xyz = "0 0 1" />
+  <origin xyz="${-1*X/2} ${Y/2} 0" rpy="0 -1.57 0" />
+</joint> -->
+<joint name="joint3" type="fixed">
+  <parent link="body" />
+  <child link="caster" />
+  <origin xyz="0 ${-1*Y/2} 0" rpy="0 -1.57 0" />
+</joint>
 </robot>

Commit message: Added plug in to gazebo xacro file

File: diff_drive/ddrive.gazebo.xacro (robot description, xacro)
@@ -1,3 +1,12 @@
 <robot name="DiffDrive" xmlns:xacro="http://www.ros.org/wiki/xacro">
+    <xacro:property name="robot_params" value = "$(find diff_drive)/config/robot_params.yaml" />
+    <xacro:property name="params" value = '${load_yaml (robot_params)}'/>
+    <xacro:property name="X" value="${params['base_x']}"/>
+    <xacro:property name="Y" value="${params['base_y']}"/>
+    <xacro:property name="Z" value="${params['base_z']}"/>
+    <xacro:property name="base_m" value="${params['base_mass']}"/>
+    <xacro:property name="r" value="${params['wheel_r']}"/>
+    <xacro:property name="l" value="${params['wheel_l']}"/>
+    <xacro:property name="wheel_m" value="${params['wheel_mass']}"/>
     <gazebo reference="body">
         <material>Gazebo/Yellow</material>
@@ -12,3 +21,25 @@
         <material>Gazebo/Blue</material>
     </gazebo>
+    <gazebo>
+        <plugin name="differential_drive_controller" filename="libgazebo_ros_diff_drive.so">
+        <rosDebugLevel>na</rosDebugLevel>
+        <alwaysOn>true</alwaysOn>
+        <updateRate>100</updateRate>
+        <leftJoint>joint2</leftJoint>
+        <rightJoint>joint1</rightJoint>
+        <wheelSeparation>${X+2*r}</wheelSeparation>
+        <wheelDiameter>${r}</wheelDiameter>
+        <wheelTorque>20</wheelTorque>
+        <commandTopic>diff/cmd_vel</commandTopic>
+        <odometryTopic>diff/odom</odometryTopic>
+        <odometryFrame>odom</odometryFrame>
+        <robotBaseFrame>base_link</robotBaseFrame>
+        <publishWheelTF>false</publishWheelTF>
+        <publishOdomTF>true</publishOdomTF>
+        <publishWheelJointState>true</publishWheelJointState>
+        <wheelAcceleration>false</wheelAcceleration>
+        <odometrySource>world</odometrySource>
+        <publishTf>1</publishTf>
+        </plugin>
+    </gazebo>
 </robot>
