Commit message: Adding gazebo set-up to launch file

File: diff_drive/ddrive.urdf.xacro (robot description, xacro)
@@ -34,9 +34,9 @@
 <joint name="joint1" type="continuous">
   <parent link="body" />
-  <child link="caster1" />
+  <child link="right_wheel" />
   <axis xyz = "0 0 1" />
   <origin xyz="0 0 ${Z/2}" rpy="0 0 0" />
 </joint>
-<link name="caster1">
+<link name="right_wheel">
   <visual>
    <inertial>
@@ -62,9 +62,9 @@
 <joint name="joint2" type="continuous">
   <parent link="body" />
-  <child link="caster2" />
+  <child link="left_wheel" />
   <axis xyz = "0 0 1" />
   <origin xyz="0 0 ${-1*Z/2}" rpy="0 0 0" />
 </joint>
-<link name="caster2">
+<link name="left_wheel">
   <visual>
    <inertial>

Commit message: Box spawns in gazebo (where are its wheels??

File: diff_drive/ddrive.urdf.xacro (robot description, xacro)
@@ -1,4 +1,5 @@
 <?xml version = "1.0"?>
 <robot name="Diff Drive" xmlns:xacro="http://www.ros.org/wiki/xacro">
+<xacro:include filename="ddrive.gazebo.xacro"/>
 <xacro:property name="robot_params" value = "$(find diff_drive)/config/robot_params.yaml" />
 <xacro:property name="params" value = '${load_yaml (robot_params)}'/>
@@ -10,4 +11,22 @@
 <xacro:property name="l" value="${params['wheel_l']}"/>
 <xacro:property name="wheel_m" value="${params['wheel_mass']}"/>
+<link name="base">
+    <visual>
+        <origin xyz="0 0 0" rpy="0 0 0"/>
+        <mass value="1"/>
+        <geometry>
+            <box size=".001 .001 .001" />
+        </geometry>
+        <material name="trans_mat">
+            <color rgba="0 0 0 0" />
+        </material>
+    </visual>
+</link>
+<joint name="fixed" type="fixed">
+  <parent link="base" />
+  <child link="body" />
+  <axis xyz = "0 0 1" />
+  <origin xyz="0 0 0" rpy="0 0 0" />
+</joint>
 <link name="body">
     <inertial>
@@ -34,9 +53,9 @@
 <joint name="joint1" type="continuous">
   <parent link="body" />
-  <child link="caster1" />
+  <child link="right_wheel" />
   <axis xyz = "0 0 1" />
-  <origin xyz="0 0 ${Z/2}" rpy="0 0 0" />
+  <origin xyz="0 ${Y/2} ${Z/2}" rpy="0 0 0" />
 </joint>
-<link name="caster1">
+<link name="right_wheel">
   <visual>
    <inertial>
@@ -45,5 +64,5 @@
      <inertia ixx="1"  ixy="1"  ixz="1" iyy="1" iyz="1" izz="1" />
    </inertial>
-   <origin xyz="0 0 ${l/2}" rpy="0 0 0" />
+   <origin xyz="0 0 ${l/2}" rpy="0 0 0"/>
    <geometry>
      <cylinder radius="${r}" length="${l}" />
@@ -54,5 +73,5 @@
   </visual>
   <collision>
-     origin xyz="0 0 ${l/2}" rpy="0 0 0" />
+    <origin xyz="0 0 ${l/2}" rpy="0 0 0"/>
    <geometry>
      <cylinder radius="${r}" length="${l}" />
@@ -62,9 +81,9 @@
 <joint name="joint2" type="continuous">
   <parent link="body" />
-  <child link="caster2" />
+  <child link="left_wheel" />
   <axis xyz = "0 0 1" />
-  <origin xyz="0 0 ${-1*Z/2}" rpy="0 0 0" />
+  <origin xyz="0 ${Y/2} ${-Z/2}" rpy="0 0 0" />
 </joint>
-<link name="caster2">
+<link name="left_wheel">
   <visual>
    <inertial>

Commit message: Attempting to make services in mover node

File: diff_drive/ddrive.urdf.xacro (robot description, xacro)
@@ -16,5 +16,5 @@
      <origin xyz="0 0 0" rpy="0 0 0"/>
      <mass value="${base_m}"/>
-     <inertia ixx="1"  ixy="1"  ixz="1" iyy="1" iyz="1" izz="1" />
+     <inertia ixx="${(base_m*(Y*Y*Z*Z))/12}"  ixy="0"  ixz="0" iyy="${(base_m*(X*X*Z*Z))/12}" iyz="0" izz="${(base_m*(X*X*Y*Y))/12}" />
     </inertial>
   <visual>
@@ -38,5 +38,5 @@
      <origin xyz="0 0 ${-1*l}" rpy="0 0 0"/>
      <mass value="${wheel_m}"/>
-     <inertia ixx="1"  ixy="1"  ixz="1" iyy="1" iyz="1" izz="1" />
+     <inertia ixx="${(wheel_m*(3*r*r+l*l))/12}"  ixy="0"  ixz="0" iyy="${(wheel_m*(3*r*r+l*l))/12}" iyz="0" izz="${(wheel_m*r*r)/2}" />
    </inertial>
   <visual>
@@ -60,5 +60,5 @@
      <origin xyz=" 0 0 ${l/2}" rpy="0 0 0"/>
      <mass value="${wheel_m}"/>
-     <inertia ixx="1"  ixy="1"  ixz="1" iyy="1" iyz="1" izz="1" />
+     <inertia ixx="${(wheel_m*(3*r*r+l*l))/12}"  ixy="0"  ixz="0" iyy="${(wheel_m*(3*r*r+l*l))/12}" iyz="0" izz="${(wheel_m*r*r)/2}" />
    </inertial>
   <visual>
@@ -82,5 +82,5 @@
      <origin xyz=" 0 0 0" rpy="0 0 0"/>
      <mass value="${wheel_m}"/>
-     <inertia ixx="1"  ixy="1"  ixz="1" iyy="1" iyz="1" izz="1" />
+     <inertia ixx="${(wheel_m*(3*Z*Z+l*l))/12}"  ixy="0"  ixz="0" iyy="${(wheel_m*(3*Z*Z+l*l))/12}" iyz="0" izz="${(wheel_m*Z*Z)/2}" />
    </inertial>
   <visual>
@@ -96,5 +96,5 @@
      <origin xyz=" 0 0 0" rpy="0 0 0"/>
    <geometry>
-    <cylinder radius="${r}" length="${l}" />
+    <cylinder radius="${Z}" length="${l}" />
    </geometry>
   </collision>

Commit message: Flippy boy

File: diff_drive/ddrive.urdf.xacro (robot description, xacro)
@@ -8,4 +8,5 @@
 <xacro:property name="Z" value="${params['base_z']}"/>
 <xacro:property name="base_m" value="${params['base_mass']}"/>
+<xacro:property name="caster_m" value="${params['caster_mass']}"/>
 <xacro:property name="r" value="${params['wheel_r']}"/>
 <xacro:property name="l" value="${params['wheel_l']}"/>
@@ -36,10 +37,10 @@
 <link name="right_wheel">
    <inertial>
-     <origin xyz="0 0 ${-1*l}" rpy="0 0 0"/>
+     <origin xyz="0 0 ${-1*l/2}" rpy="0 0 0"/>
      <mass value="${wheel_m}"/>
      <inertia ixx="${(wheel_m*(3*r*r+l*l))/12}"  ixy="0"  ixz="0" iyy="${(wheel_m*(3*r*r+l*l))/12}" iyz="0" izz="${(wheel_m*r*r)/2}" />
    </inertial>
   <visual>
-   <origin xyz="0 0 ${-1*l}" rpy="0 0 0"/>
+   <origin xyz="0 0 ${-1*l/2}" rpy="0 0 0"/>
    <geometry>
      <cylinder radius="${r}" length="${l}" />
@@ -50,5 +51,5 @@
   </visual>
   <collision>
-   <origin xyz="0 0 ${-1*l}" rpy="0 0 0"/>
+   <origin xyz="0 0 ${-1*l/2}" rpy="0 0 0"/>
    <geometry>
      <cylinder radius="${r}" length="${l}" />
@@ -81,6 +82,6 @@
    <inertial>
      <origin xyz=" 0 0 0" rpy="0 0 0"/>
-     <mass value="${wheel_m}"/>
-     <inertia ixx="${(wheel_m*(3*Z*Z+l*l))/12}"  ixy="0"  ixz="0" iyy="${(wheel_m*(3*Z*Z+l*l))/12}" iyz="0" izz="${(wheel_m*Z*Z)/2}" />
+     <mass value="${caster_m}"/>
+     <inertia ixx="${(caster_m*(3*Z*Z+l*l))/12}"  ixy="0"  ixz="0" iyy="${(caster_m*(3*Z*Z+l*l))/12}" iyz="0" izz="${(caster_m*Z*Z)/2}" />
    </inertial>
   <visual>
